File: STM32F103ZET6/STM32F103ZET6.sch (KiCad schematic (older format))
At the start: 1 part, among them U1 STM32F103ZETx

Commit message: Update STM32F103ZET6.sch
Parts:
- added C1, C2: 6pF, symbol Device:C
- added C3, C4: 22pF, symbol Device:C
- added C5: 104, symbol Device:C
- added R1: 20M, symbol Device:R
- added R2, R3, R4: 10K, symbol Device:R
- added SW1: RESET, symbol Switch:SW_Push_Dual
- added Y1: 32.768KHz, symbol Device:Crystal
- added Y2: 8MHz, symbol Device:Crystal
Connections:
- net labels added: BOOT0, BOOT1, GND, NRST, VDD
- wire segments 0 -> 52
Other:
- note added: "32.768MHz Oscillator"
- note added: "8MHz Oscillator"
- note added: "Boot configuration"
- note added: "MCU\n"
- note added: "Reset\n"

Commit message: adjust MCU position
Connections:
- net labels added: OSC_32.768KHz_IN, OSC_32.768KHz_OUT, OSC_8MHz_IN, OSC_8MHz_OUT
Other:
- moved on the sheet: C1, C2, C3, C4, C5, R1, R2, R3, R4, SW1, U1, Y1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

Commit message: fix net label
Other:
- note added: "32.768KHz Oscillator"
- note removed: "32.768MHz Oscillator"
Changed lines of the file:
@@
 8MHz Oscillator
 Text Notes 15550 13100 0    79   ~ 0
-32.768MHz Oscillator
+32.768KHz Oscillator
 $Comp
 L Device:R R3
@@
 Text Label 11300 12250 0    50   ~ 0
 OSC_8MHz_IN
-Text Label 10400 5800 2    79   ~ 0
+Text Label 10400 5800 2    50   ~ 0
 OSC_32.768KHz_IN
-Text Label 10400 5700 2    79   ~ 0
+Text Label 10400 5700 2    50   ~ 0
 OSC_32.768KHz_OUT
 Wire Wire Line

Commit message: update
Parts:
- added BT?: Battery_Cell, symbol Device:Battery_Cell
- added C? (x2): C, symbol Device:C
- added C? (x11): 104, symbol Device:C
- added L?: L, symbol Device:L
Connections:
- net labels added: +3.3V, VBAT, VDD1, VDD10, VDD11, VDD2, VDD3, VDD4, VDD5, VDD6, VDD7, VDD8, VDD9, VDDA, VREF+, VREF-, VSS1, VSS10, VSS11, VSS2, VSS3, VSS4, VSS5, VSS6, VSS7, VSS8, VSS9, VSSA
- wire segments 52 -> 97
Other:
- note added: "MCU POWER"
- moved on the sheet: C1, C2, C3, C4, C5, R1, R2, R3, R4, SW1, U1, Y1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

Commit message: update
Parts:
- added C19: 220uF, symbol Device:C
- added C20, C21, C22, C25: 104, symbol Device:C
- added C23: 10uF, symbol Device:C
- added C24: 100uF, symbol Device:C
- added D1, D4: 1N5822, Diode_THT:D_DO-201AD_P15.24mm_Horizontal, symbol Diode:1N5822
- added D2: SMAJ 5.0A, Diode_THT:D_DO-201AD_P15.24mm_Horizontal, symbol Diode:1N5822
- added D3: LED, symbol Device:LED
- added F1: Fuse, symbol Device:Fuse
- added J1: Conn_01x02_Female, symbol Connector:Conn_01x02_Female
- added J2: Jack-DC, symbol Connector:Jack-DC
- added L2: 33uH, symbol Device:L_Core_Iron
- added R5: 1k, symbol Device:R
- added SW2: SW_DIP_x01, symbol Switch:SW_DIP_x01
- added U2: LM2596S-5, Package_TO_SOT_SMD:TO-263-5_TabPin3, symbol Regulator_Switching:LM2596S-5
- added U3: AMS1117-3.3, Package_TO_SOT_SMD:SOT-223-3_TabPin2, symbol Regulator_Linear:AMS1117-3.3
- gave numbers to parts that had none: 15
Connections:
- net labels added: +12V, +5V
- wire segments 97 -> 162
Other:
- note added: "3.3 Voltage Regulator"
- note added: "5 Voltage Regulator"

Commit message: add 74HC1G66GW to schematic
Parts:
- removed J1: Conn_01x02_Female, symbol Connector:Conn_01x02_Female
- added 1M1, R10, R6, R7, R8, R9: R, symbol Device:R
- added C26, C29: 104, symbol Device:C
- added C27: 10uF, symbol Device:CP
- added C28, C30: 22pF, symbol Device:C
- added C31, C32: C, symbol Device:C
- added D5: 1N4148, Diode_THT:D_DO-35_SOD27_P7.62mm_Horizontal, symbol Diode:1N4148
- added IC1: 74HC1G66GW, SOT65P212X110-5N, symbol 74HC1G66GW_125:74HC1G66GW,125
- added J1: Conn_01x02, symbol Connector_Generic:Conn_01x02
- added J3, J4, J5: +5V, symbol Connector_Generic:Conn_01x01
- added J6: USB_B_Micro, symbol Connector:USB_B_Micro
- added JP1, JP2: Jumper_NO_Small, symbol Device:Jumper_NO_Small
- added Q1: S8050, Package_TO_SOT_THT:TO-92_Inline, symbol Transistor_BJT:S8050
- added Q2: S8550, Package_TO_SOT_THT:TO-92_Inline, symbol Transistor_BJT:S8550
- added U4: CH340G, Package_SO:SOIC-16_3.9x9.9mm_P1.27mm, symbol Interface_USB:CH340G
- added Y3: 12MHz, symbol Device:Crystal
- D2: value SMAJ 5.0A -> SMAJ5.0A
- L1: value L -> BLM18PG181SN1D
- U2: value LM2596S-5 -> LM2596S-5.0
Connections:
- net labels added: DTR, Earth, RESET, RTS, USART1_RXD, USART1_TXD, USB_5V, VCC_3V3
- wire segments 162 -> 225
- no-connect marks 0 -> 5
Other:
- note added: "ISP"
- moved on the sheet: C10, C11, C12, C15, C16, C17, C18, C21, C22, C23, C6, C7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

Commit message: add net label
Parts:
- removed J4, J5: +5V, symbol Connector_Generic:Conn_01x01
- added R?: 1k, symbol Device:R
- C32: value C -> 22uF
- R10: value R -> 100k
- R6, R8, R9: value R -> 1k
- R7: value R -> 10k
Connections:
- net labels added: EXT_5V, VCC_3.3V, VCC_5V
- net labels removed: +3.3V, +5V
- wire segments 225 -> 228
Other:
- moved on the sheet: 1M1, C26, C27, C28, C29, C30, C31, C32, D5, F1, IC1, J6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

Commit message: update schematic
Parts:
- added J?: Conn_01x06, symbol Connector_Generic:Conn_01x06
- added R? (x2): R, symbol Device:R
Connections:
- net labels added: JTCK\SWCLK, JTDO\SWO, JTMS\SWDIO
- net labels removed: NRST
- wire segments 228 -> 243
Other:
- note added: "STLink"
Changed lines of the file:
@@
 	10950 15500 10650 15500
 Text Label 3550 15500 0    50   ~ 0
-NRST
+RESET
 Wire Wire Line
 	6900 15350 6900 15500
@@
 BOOT0
 Wire Notes Line
-	13000 3000 22900 3000
+	13000 2950 22900 2950
 Wire Wire Line
 	20300 1600 20300 1800
@@
 Wire Wire Line
 	18700 1950 19750 1950
+$Comp
+L Connector_Generic:Conn_01x06 J?
+U 1 1 5E52456F
+P 21850 3900
+F 0 "J?" H 21930 3892 50  0000 L CNN
+F 1 "Conn_01x06" H 21930 3801 50  0000 L CNN
+F 2 "" H 21850 3900 50  0001 C CNN
+F 3 "~" H 21850 3900 50  0001 C CNN
+	1    21850 3900
+	1    0    0    -1
+$EndComp
+Wire Wire Line
+	21650 3700 20550 3700
+Wire Wire Line
+	21650 3800 21150 3800
+Wire Wire Line
+	21650 3900 20850 3900
+Wire Wire Line
+	21650 4000 20550 4000
+Wire Wire Line
+	21350 4100 21650 4100
+Text Label 21350 4100 2    50   ~ 0
+VCC_3V3
+$Comp
+L power:GND #PWR?
+U 1 1 5E58D437
+P 21550 4200
+F 0 "#PWR?" H 21550 3950 50  0001 C CNN
+F 1 "GND" H 21555 4027 50  0000 C CNN
+F 2 "" H 21550 4200 50  0001 C CNN
+F 3 "" H 21550 4200 50  0001 C CNN
+	1    21550 4200
+	1    0    0    -1
+$EndComp
+Wire Wire Line
+	21550 4200 21650 4200
+$Comp
+L Device:R R?
+U 1 1 5E59CB21
+P 20850 3450
+F 0 "R?" H 20920 3496 50  0000 L CNN
+F 1 "R" H 20920 3405 50  0000 L CNN
+F 2 "" V 20780 3450 50  0001 C CNN
+F 3 "~" H 20850 3450 50  0001 C CNN
+	1    20850 3450
+	1    0    0    -1
+$EndComp
+$Comp
+L Device:R R?
+U 1 1 5E5A9CA3
+P 21150 3450
+F 0 "R?" H 21220 3496 50  0000 L CNN
+F 1 "R" H 21220 3405 50  0000 L CNN
+F 2 "" V 21080 3450 50  0001 C CNN
+F 3 "~" H 21150 3450 50  0001 C CNN
+	1    21150 3450
+	1    0    0    -1
+$EndComp
+Connection ~ 20850 3900
+Wire Wire Line
+	20850 3900 20550 3900
+Wire Wire Line
+	20850 3200 21000 3200
+Connection ~ 21150 3800
+Wire Wire Line
+	20550 3800 21150 3800
+Connection ~ 21000 3200
+Wire Wire Line
+	21000 3200 21150 3200
+Text Label 21000 3100 0    50   ~ 0
+VCC_3V3
+Text Label 20550 3700 2    50   ~ 0
+JTCK\SWCLK
+Text Label 20550 3800 2    50   ~ 0
+JTMS\SWDIO
+Text Label 20550 3900 2    50   ~ 0
+JTDO\SWO
+Text Label 20550 4000 2    50   ~ 0
+RESET
+Wire Wire Line
+	20850 3600 20850 3900
+Wire Wire Line
+	21150 3600 21150 3800
+Wire Wire Line
+	20850 3200 20850 3300
+Wire Wire Line
+	21150 3200 21150 3300
+Wire Wire Line
+	21000 3100 21000 3200
+Text Label 10200 6850 1    50   ~ 0
+JTCK\SWCLK
+Text Label 10300 6850 1    50   ~ 0
+JTMS\SWDIO
+Text Label 10800 6850 1    50   ~ 0
+JTDO\SWO
+Wire Notes Line
+	22900 4550 19750 4550
+Wire Notes Line
+	19750 4550 19750 2950
+Text Label 8800 9450 3    50   ~ 0
+RESET
+Text Notes 22350 4350 0    79   ~ 0
+STLink
 Wire Bus Line
 	3600 800  3600 2000
